File: Hover Copters.sch (KiCad schematic (older format))
At the start: 26 parts, among them J1 Angle POT, J2 +5V_IN, J3 Motor, J4 Shaft_Angle_Encoder, J5 5V or your voltage, Q1 PZT2222A, Q2 D45H11, U1 ESP32-DEVKITC-32D

Commit message: Note about fixing the IO0 being pulled up.
Parts:
- U1: symbol ESP32-DEVKITC-32D:ESP32-DEVKITC-32D -> Hover-Copters-rescue:ESP32-DEVKITC-32D-ESP32-DEVKITC-32D
Other:
- note added: "Move the IO pins to IO18 and IO19 for the shaft angle encoder."
Changed lines of the file:
@@
 $EndDescr
 $Comp
-L ESP32-DEVKITC-32D:ESP32-DEVKITC-32D U1
+L Hover-Copters-rescue:ESP32-DEVKITC-32D-ESP32-DEVKITC-32D U1
 U 1 1 60528A5A
 P 5450 3300
@@
 Wire Wire Line
 	3050 4050 2950 4050
+Text Notes 5700 4500 0    50   ~ 0
+Move the IO pins to IO18 and IO19 for the shaft angle encoder.
 $EndSCHEMATC

Commit message: Added encoder datasheet.
Parts:
- J4: Encoder Data (none) -> https://cdn.automationdirect.com/static/specs/encoderld.pdf
Changed lines of the file:
@@
 F 2 "Connector_PinHeader_2.54mm:PinHeader_1x04_P2.54mm_Vertical" H 2750 3950 50  0001 C CNN
 F 3 "https://www.te.com/usa-en/products/connectors/pcb-connectors/intersection/mta-100-mta-156-connectors.html?tab=pgp-story" H 2750 3950 50  0001 C CNN
+F 4 "https://cdn.automationdirect.com/static/specs/encoderld.pdf" H 2750 3950 50  0001 C CNN "Encoder Data"
 	1    2750 3950
 	1    0    0    -1
